File: USBTTL.kicad_sch (KiCad schematic)
At the start: 22 parts, among them J1 USB_C_Receptacle_USB2.0, J2 Conn_01x06_Female, J3 Conn_01x06_Male, SW1 SW_DPDT_x2, SW2 SW_DPDT_x2, U1 FT231XS

Commit message: Finish wiring.
Parts:
- removed SW1, SW2: SW_DPDT_x2, symbol Switch:SW_DPDT_x2
- added R8: 0, Resistor_SMD:R_0603_1608Metric_Pad0.98x0.95mm_HandSolder, symbol Device:R
- added SW1, SW2: SW_SPDT, Button_Switch_SMD:SW_SPDT_PCM12, symbol Switch:SW_SPDT
- C1, C2, C3, C4, C5, C6: footprint (none) -> Capacitor_SMD:C_0603_1608Metric_Pad1.08x0.95mm_HandSolder
- D1: footprint (none) -> LED_SMD:LED_0603_1608Metric_Pad1.05x0.95mm_HandSolder
- J1: footprint (none) -> Connector_USB:USB_C_Receptacle_Palconn_UTC16-G
- J2: footprint (none) -> Connector_PinSocket_2.54mm:PinSocket_1x06_P2.54mm_Vertical
- J3: footprint (none) -> Connector_PinHeader_2.54mm:PinHeader_1x06_P2.54mm_Horizontal
- R1, R2, R3, R4, R5, R6, R7: footprint (none) -> Resistor_SMD:R_0603_1608Metric_Pad0.98x0.95mm_HandSolder
- RX1: renamed from RXLED1; footprint (none) -> LED_SMD:LED_0603_1608Metric_Pad1.05x0.95mm_HandSolder
- TX1: renamed from TXLED1; footprint (none) -> LED_SMD:LED_0603_1608Metric_Pad1.05x0.95mm_HandSolder
Connections:
- net +3V3: now also SW1.3 (C)
- net +5V: now also J2.6 (Pin_6), J3.6 (Pin_6), SW1.1 (A); no longer J2.1 (Pin_1), J3.1 (Pin_1)
- net GND: now also J2.1 (Pin_1), J3.1 (Pin_1); no longer J2.6 (Pin_6), J3.6 (Pin_6)
- net IOLEVEL: now also R8.2
- net PINSEL: now also SW2.2 (B)
- net RX: now also J2.4 (Pin_4), J3.4 (Pin_4); no longer J2.5 (Pin_5), J3.5 (Pin_5)
- net TX: now also J2.5 (Pin_5), J3.5 (Pin_5); no longer J2.4 (Pin_4), J3.4 (Pin_4)
- net ~{CTS}: now also SW2.1 (A)
- net ~{RTS}: now also SW2.3 (C)
- net USBD+: now reaches R4.2, U1.11 (USBDP)
- net USBD-: now reaches R3.2, U1.12 (USBDM)
- new net: R8.1, SW1.2 (B)
